Commit message: Update ManiSkill2_real2sim

File: data/custom/mk_station_original.urdf (robot description, URDF)
Before this commit: robot mk_station, 4 links, 3 joints
Links:
- removed link body
- removed link bottom_drawer
- removed link top_drawer
- added link body1; collision box size=0.02000 0.61500 0.84500; collision box size=0.59000 0.02000 0.84500
- added link body2; collision box size=0.02000 0.61500 0.84500; collision box size=0.59000 0.02000 0.84500
- added link bottom_drawer1; collision box size=0.015000 0.61500 0.14000; collision box size=0.02000 0.51500 0.10000
- added link bottom_drawer2; collision box size=0.015000 0.61500 0.14000; collision box size=0.02000 0.51500 0.10000
- added link top_drawer1; collision box size=0.015000 0.61500 0.14000; collision box size=0.02000 0.51500 0.10000
Joints:
- removed joint bottom_drawer_joint
- removed joint top_drawer_joint
- added joint bottom_drawer1_joint: type prismatic, parent body1, child bottom_drawer1, origin xyz=0.00000 0.00000 0.17800 rpy=0.00000 0.00000 0.00000, axis 1.00000 0.00000 0.00000, limit lower=0 upper=0.5 effort=0.00000 velocity=0.00000
- added joint bottom_drawer2_joint: type prismatic, parent body2, child bottom_drawer2, origin xyz=0.00000 0.10000 0.17800 rpy=0.00000 0.00000 0.00000, axis 1.00000 0.00000 0.00000, limit lower=0 upper=0.5 effort=0.00000 velocity=0.00000
- added joint middle_drawer2_joint: type prismatic, parent body2, child middle_drawer2, origin xyz=0.00000 0.10000 0.42300 rpy=0.00000 0.00000 0.00000, axis 1.00000 0.00000 0.00000, limit lower=0 upper=0.5 effort=0.00000 velocity=0.00000
- added joint top_drawer1_joint: type prismatic, parent body1, child top_drawer1, origin xyz=0.00000 0.00000 0.66800 rpy=0.00000 0.00000 0.00000, axis 1.00000 0.00000 0.00000, limit lower=0 upper=0.5 effort=0.00000 velocity=0.00000
- added joint top_drawer2_joint: type prismatic, parent body2, child top_drawer2, origin xyz=0.00000 0.10000 0.66800 rpy=0.00000 0.00000 0.00000, axis 1.00000 0.00000 0.00000, limit lower=0 upper=0.5 effort=0.00000 velocity=0.00000
- joint middle_drawer_joint: parent body -> body1
