Commit message: Update ManiSkill2_real2sim submodule

File: data/custom/mk_station_v1.urdf (robot description, URDF)
Before this commit: robot mk_station, 4 links, 3 joints
Links:
- removed link middle_drawer
- link bottom_drawer: geometry collision box size=0.015000 0.61500 0.14000; collision box size=0.02000 0.51500 0.10000
Joints:
- removed joint middle_drawer_joint

File: data/custom/mk_station_v2.urdf (robot description, URDF)
Before this commit: robot mk_station, 4 links, 3 joints
Links:
- removed link middle_drawer
- link bottom_drawer: geometry collision box size=0.015000 0.61500 0.25000; collision box size=0.02000 0.51500 0.10000
- link top_drawer: geometry collision box size=0.015000 0.61500 0.3000; collision box size=0.02000 0.51500 0.20000
Joints:
- removed joint middle_drawer_joint
